File: NGL_PCB/NGL_PCB.sch (KiCad schematic (older format))
At the start: 126 parts, among them U11 TL064, U12 TL064, U13 TL064, U14 TL064, U15 TL064, U21 TL064, U22 TL064, U23 TL064, U24 TL064, U25 TL064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

Commit message: MOD AU 03/02
Connections:
- net at D2.1 (K), D3.2 (A), D4.1 (K)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: now also D1.2 (A), R2.2
- net at U13.9 (-): now also R3.2, R4.2, R6.1
- net at R31.2, U9.5 (VOUT): no longer C18.2, VT3.2 (E)
- net S0: now reaches U6.10 (S0)
- net S1: now reaches U6.9 (S1)
- new net: C18.2, VT3.2 (E)
Other:
- moved on the sheet: C16, C18, C33, C34, C4, C5, C7, C8, C?, D2, D4, L2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
